Commit message: migration to windows

File: VENV/urdf/iCook.urdf (robot description, URDF)
Before this commit: robot mrm, 6 links, 5 joints
Joints:
- joint base_link_to_link_1: limit lower=-3.14 upper=3.14 effort=1000.0 velocity=0.5 -> lower=-1.57 upper=1.57 effort=1000.0 velocity=0.5
- joint link_1_to_link_2: limit lower=-3.14 upper=3.14 effort=1000.0 velocity=0.5 -> lower=-1.57 upper=1.57 effort=1000.0 velocity=0.5
- joint link_2_to_link_3: limit lower=-3.14 upper=3.14 effort=1000.0 velocity=0.5 -> lower=-1.57 upper=1.57 effort=1000.0 velocity=0.5
- joint link_3_to_link_4: limit lower=-3.14 upper=3.14 effort=1000.0 velocity=0.5 -> lower=-1.57 upper=1.57 effort=1000.0 velocity=0.5
- joint link_4_to_link_5: limit lower=-3.14 upper=3.14 effort=1000.0 velocity=0.5 -> lower=-1.57 upper=1.57 effort=1000.0 velocity=0.5
